File: Плата датчиков.kicad_pcb (KiCad board)
At the start: 4 copper layers, 67 x 68.5 mm, 51 parts, among them J1 A, J10 4900, J11 4900, J12 4900, J14 4900, J2 B, J3 C, J4 Conn_02x07_Odd_Even, J5 4900, J6 4900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

Commit message: Финальная доработка
Parts:
- moved R10 4.77 mm to (79.8, 110.2)
- moved R11 4.77 mm to (76.2, 110.2)
- moved R12 4.77 mm to (74.4, 110.2)
- moved R13 4.77 mm to (75.7, 122.6)
- moved R14 4.77 mm to (73.2, 122.6)
- moved R9 4.77 mm to (78.0, 110.2)
- moved U4 4.77 mm to (77.0, 116.8)
- moved C10 4.75 mm to (78.0, 110.2)
- moved C11 4.75 mm to (79.8, 110.2)
- moved C12 4.75 mm to (76.2, 110.2)
- moved C13 4.75 mm to (74.4, 110.2)
- moved C14 4.75 mm to (75.7, 122.7)
- moved C17 4.75 mm to (73.2, 122.7)
- moved C18 4.75 mm to (77.0, 116.9)
- turned J8 to -45 degrees
Changed lines of the file:
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@@
   )
   (footprint "Resistor_SMD:R_0603_1608Metric_Pad0.98x0.95mm_HandSolder" (layer "F.Cu")
-    (at 78.994 111.5415 -90)
+    (at 74.422 110.171 -90)
     (descr "Resistor SMD 0603 (1608 Metric), square (rectangular) end terminal, IPC_7351 nominal with elongated pad for handsoldering. (Body size source: IPC-SM-782 page 72, https://www.pcb-3d.com/wordpress/wp-content/uploads/ipc-sm-782a_amendment_1_and_2.pdf), generated with kicad-footprint-generator")
     (tags "resistor handsolder")
@@
   )
   (footprint "Resistor_SMD:R_0603_1608Metric_Pad0.98x0.95mm_HandSolder" (layer "F.Cu")
-    (at 84.328 111.5415 -90)
+    (at 79.756 110.171 -90)
     (descr "Resistor SMD 0603 (1608 Metric), square (rectangular) end terminal, IPC_7351 nominal with elongated pad for handsoldering. (Body size source: IPC-SM-782 page 72, https://www.pcb-3d.com/wordpress/wp-content/uploads/ipc-sm-782a_amendment_1_and_2.pdf), generated with kicad-footprint-generator")
     (tags "resistor handsolder")
@@
   )
   (footprint "Resistor_SMD:R_0603_1608Metric_Pad0.98x0.95mm_HandSolder" (layer "F.Cu")
-    (at 80.772 111.5415 -90)
+    (at 76.2 110.171 -90)
     (descr "Resistor SMD 0603 (1608 Metric), square (rectangular) end terminal, IPC_7351 nominal with elongated pad for handsoldering. (Body size source: IPC-SM-782 page 72, https://www.pcb-3d.com/wordpress/wp-content/uploads/ipc-sm-782a_amendment_1_and_2.pdf), generated with kicad-footprint-generator")
     (tags "resistor handsolder")
@@
   )
   (footprint "Package_SO:SOIC-14_3.9x8.7mm_P1.27mm" (layer "F.Cu")
-    (at 81.534 118.2105 -90)
+    (at 76.962 116.84 -90)
     (descr "SOIC, 14 Pin (JEDEC MS-012AB, https://www.analog.com/media/en/package-pcb-resources/package/pkg_pdf/soic_narrow-r/r_14.pdf), generated with kicad-footprint-generator ipc_gullwing_generator.py")
     (tags "SOIC SO")
@@
   )
   (footprint "Resistor_SMD:R_0603_1608Metric_Pad0.98x0.95mm_HandSolder" (layer "F.Cu")
-    (at 82.55 111.5415 -90)
+    (at 77.978 110.171 -90)
     (descr "Resistor SMD 0603 (1608 Metric), square (rectangular) end terminal, IPC_7351 nominal with elongated pad for handsoldering. (Body size source: IPC-SM-782 page 72, https://www.pcb-3d.com/wordpress/wp-content/uploads/ipc-sm-782a_amendment_1_and_2.pdf), generated with kicad-footprint-generator")
     (tags "resistor handsolder")
@@
   )
   (footprint "Resistor_SMD:R_0603_1608Metric_Pad0.98x0.95mm_HandSolder" (layer "F.Cu")
-    (at 77.724 123.9875 90)
+    (at 73.152 122.617 90)
     (descr "Resistor SMD 0603 (1608 Metric), square (rectangular) end terminal, IPC_7351 nominal with elongated pad for handsoldering. (Body size source: IPC-SM-782 page 72, https://www.pcb-3d.com/wordpress/wp-content/uploads/ipc-sm-782a_amendment_1_and_2.pdf), generated with kicad-footprint-generator")
     (tags "resistor handsolder")
@@
   )
   (footprint "Connector_PinHeader_2.54mm:PinHeader_2x02_P2.54mm_Vertical" (layer "F.Cu")
-    (at 67 110)
+    (at 67 110 -45)
     (descr "Through hole straight pin header, 2x02, 2.54mm pitch, double rows")
     (tags "Through hole pin header THT 2x02 2.54mm double row")
@@
     (property "Поле2" "")
     (attr through_hole)
-    (fp_text reference "J8" (at 1.27 -2.33) (layer "F.SilkS")
-        (effects (font (size 1 1) (thickness 0.15)))
-    )
-    (fp_text value "Conn_02x02_Odd_Even" (at 1.27 4.87) (layer "F.Fab")
-        (effects (font (size 1 1) (thickness 0.15)))
-    )
-    (fp_text user "${REFERENCE}" (at 1.27 1.27 90) (layer "F.Fab")
+    (fp_text reference "J8" (at 1.27 -2.33 135) (layer "F.SilkS")
+        (effects (font (size 1 1) (thickness 0.15)))
+    )
+    (fp_text value "Conn_02x02_Odd_Even" (at 1.27 4.87 135) (layer "F.Fab")
+        (effects (font (size 1 1) (thickness 0.15)))
+    )
+    (fp_text user "${REFERENCE}" (at 1.27 1.27 45) (layer "F.Fab")
         (effects (font (size 1 1) (thickness 0.15)))
     )
@@
     (fp_line (start 3.81 3.81) (end -1.27 3.81)
       (stroke (width 0.1) (type solid)) (layer "F.Fab"))
-    (pad "1" thru_hole rect (at 0 0) (size 1.7 1.7) (drill 1) (layers "*.Cu" "*.Mask")
+    (pad "1" thru_hole rect (at 0 0 315) (size 1.7 1.7) (drill 1) (layers "*.Cu" "*.Mask")
       (net 31 "PTC_Coil_A") (pinfunction "Pin_1") (pintype "passive"))
-    (pad "2" thru_hole oval (at 2.54 0) (size 1.7 1.7) (drill 1) (layers "*.Cu" "*.Mask")
+    (pad "2" thru_hole oval (at 2.54 0 315) (size 1.7 1.7) (drill 1) (layers "*.Cu" "*.Mask")
       (net 36 "PTC_Coil_C") (pinfunction "Pin_2") (pintype "passive"))
-    (pad "3" thru_hole oval (at 0 2.54) (size 1.7 1.7) (drill 1) (layers "*.Cu" "*.Mask")
+    (pad "3" thru_hole oval (at 0 2.54 315) (size 1.7 1.7) (drill 1) (layers "*.Cu" "*.Mask")
       (net 35 "PTC_Coil_B") (pinfunction "Pin_3") (pintype "passive"))
-    (pad "4" thru_hole oval (at 2.54 2.54) (size 1.7 1.7) (drill 1) (layers "*.Cu" "*.Mask")
+    (pad "4" thru_hole oval (at 2.54 2.54 315) (size 1.7 1.7) (drill 1) (layers "*.Cu" "*.Mask")
       (net 26 "GNDA") (pinfunction "Pin_4") (pintype "passive"))
     (model "${KICAD6_3DMODEL_DIR}/Connector_PinHeader_2.54mm.3dshapes/PinHeader_2x02_P2.54mm_Vertical.step"
@@
   )
   (footprint "Resistor_SMD:R_0603_1608Metric_Pad0.98x0.95mm_HandSolder" (layer "F.Cu")
-    (at 80.264 123.9875 90)
+    (at 75.692 122.617 90)
     (descr "Resistor SMD 0603 (1608 Metric), square (rectangular) end terminal, IPC_7351 nominal with elongated pad for handsoldering. (Body size source: IPC-SM-782 page 72, https://www.pcb-3d.com/wordpress/wp-content/uploads/ipc-sm-782a_amendment_1_and_2.pdf), generated with kicad-footprint-generator")
     (tags "resistor handsolder")
@@
   )
   (footprint "Capacitor_SMD:C_0603_1608Metric_Pad1.08x0.95mm_HandSolder" (layer "B.Cu")
-    (at 82.55 111.5415 90)
+    (at 77.978 110.236 90)
     (descr "Capacitor SMD 0603 (1608 Metric), square (rectangular) end terminal, IPC_7351 nominal with elongated pad for handsoldering. (Body size source: IPC-SM-782 page 76, https://www.pcb-3d.com/wordpress/wp-content/uploads/ipc-sm-782a_amendment_1_and_2.pdf), generated with kicad-footprint-generator")
     (tags "capacitor handsolder")
@@
   )
   (footprint "Capacitor_SMD:C_0603_1608Metric_Pad1.08x0.95mm_HandSolder" (layer "B.Cu")
-    (at 78.994 111.5415 -90)
+    (at 74.422 110.236 -90)
     (descr "Capacitor SMD 0603 (1608 Metric), square (rectangular) end terminal, IPC_7351 nominal with elongated pad for handsoldering. (Body size source: IPC-SM-782 page 76, https://www.pcb-3d.com/wordpress/wp-content/uploads/ipc-sm-782a_amendment_1_and_2.pdf), generated with kicad-footprint-generator")
     (tags "capacitor handsolder")
@@
   )
   (footprint "Capacitor_SMD:C_0603_1608Metric_Pad1.08x0.95mm_HandSolder" (layer "B.Cu")
-    (at 77.724 123.9875 90)
+    (at 73.152 122.682 90)
     (descr "Capacitor SMD 0603 (1608 Metric), square (rectangular) end terminal, IPC_7351 nominal with elongated pad for handsoldering. (Body size source: IPC-SM-782 page 76, https://www.pcb-3d.com/wordpress/wp-content/uploads/ipc-sm-782a_amendment_1_and_2.pdf), generated with kicad-footprint-generator")
     (tags "capacitor handsolder")
@@
   )
   (footprint "Capacitor_SMD:C_0603_1608Metric_Pad1.08x0.95mm_HandSolder" (layer "B.Cu")
-    (at 80.264 123.9875 -90)
+    (at 75.692 122.682 -90)
     (descr "Capacitor SMD 0603 (1608 Metric), square (rectangular) end terminal, IPC_7351 nominal with elongated pad for handsoldering. (Body size source: IPC-SM-782 page 76, https://www.pcb-3d.com/wordpress/wp-content/uploads/ipc-sm-782a_amendment_1_and_2.pdf), generated with kicad-footprint-generator")
     (tags "capacitor handsolder")
@@
   )
   (footprint "Capacitor_SMD:C_0603_1608Metric_Pad1.08x0.95mm_HandSolder" (layer "B.Cu")
-    (at 84.328 111.5415 -90)
+    (at 79.756 110.236 -90)
     (descr "Capacitor SMD 0603 (1608 Metric), square (rectangular) end terminal, IPC_7351 nominal with elongated pad for handsoldering. (Body size source: IPC-SM-782 page 76, https://www.pcb-3d.com/wordpress/wp-content/uploads/ipc-sm-782a_amendment_1_and_2.pdf), generated with kicad-footprint-generator")
     (tags "capacitor handsolder")
@@
   )
   (footprint "Capacitor_SMD:C_0603_1608Metric_Pad1.08x0.95mm_HandSolder" (layer "B.Cu")
-    (at 81.534 118.2105 -90)
+    (at 76.962 116.905 -90)
     (descr "Capacitor SMD 0603 (1608 Metric), square (rectangular) end terminal, IPC_7351 nominal with elongated pad for handsoldering. (Body size source: IPC-SM-782 page 76, https://www.pcb-3d.com/wordpress/wp-content/uploads/ipc-sm-782a_amendment_1_and_2.pdf), generated with kicad-footprint-generator")
     (tags "capacitor handsolder")
@@
   )
   (footprint "Capacitor_SMD:C_0603_1608Metric_Pad1.08x0.95mm_HandSolder" (layer "B.Cu")
-    (at 80.772 111.5415 90)
+    (at 76.2 110.236 90)
     (descr "Capacitor SMD 0603 (1608 Metric), square (rectangular) end terminal, IPC_7351 nominal with elongated pad for handsoldering. (Body size source: IPC-SM-782 page 76, https://www.pcb-3d.com/wordpress/wp-content/uploads/ipc-sm-782a_amendment_1_and_2.pdf), generated with kicad-footprint-generator")
     (tags "capacitor handsolder")

Commit message: Ещё доработать
Parts:
- C15: moved to B.Cu
- C7, C8, R5, R6, U2: moved to F.Cu
- moved J10 43.8 mm to (71.9, 117.7)
- moved J8 43.3 mm to (97.8, 79.5), turned to 135 degrees
- moved J7 42.8 mm to (76.7, 120.1), turned to 70 degrees
- moved J11 42.6 mm to (67.5, 114.7), turned to 50 degrees
- moved C17 41.7 mm to (85.3, 82.8), turned to 0 degrees
- moved R14 41.7 mm to (85.4, 82.8), turned to 0 degrees
- moved C14 38.6 mm to (85.3, 85.3), turned to 180 degrees
- moved R13 38.5 mm to (85.4, 85.3), turned to 0 degrees
- moved R12 35.1 mm to (97.9, 84.1), turned to 180 degrees
- moved C18 33.4 mm to (91.1, 86.6), turned to 180 degrees
- moved U4 33.4 mm to (91.2, 86.6), turned to 180 degrees
- moved R11 32.6 mm to (97.9, 85.9), turned to 180 degrees
- moved C13 31.9 mm to (91.2, 83.1), turned to 180 degrees
- moved R9 30.1 mm to (97.9, 87.6), turned to 180 degrees
- moved C12 29.5 mm to (91.2, 84.8), turned to 180 degrees
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- renumbered Je to J13
Connections:
- C4 pad 2: Net-(D1-OUT) -> OUT_MCU
- D1 pad 3: Net-(D1-OUT) -> OUT_MCU
- J10 pad 1: B_OUT -> C_OUT
- J10 pad 2: B_OUT -> C_OUT
- J11 pad 1: B_OUT -> C_OUT
- J11 pad 2: B_OUT -> C_OUT
- J12 pad 1: C_OUT -> B_OUT
- J12 pad 2: C_OUT -> B_OUT
- J13 pad 1: C_OUT -> B_OUT
- J13 pad 2: C_OUT -> B_OUT
- J14 pad 1: C_OUT -> B_OUT
- J14 pad 2: C_OUT -> B_OUT
- J4 pad 10: Temp_Coil_A_MCU -> Current_C_MCU
- J4 pad 3: SCLK_MCU -> CS_MCU
- J4 pad 4: GNDA -> Temp_Coil_C_MCU
- J4 pad 5: CS_MCU -> SCLK_MCU
- J4 pad 6: Temp_Coil_C_MCU -> Temp_Coil_B_MCU
- J4 pad 8: Temp_Coil_B_MCU -> Temp_Coil_A_MCU
- J4 pad 9: Current_C_MCU -> OUT_MCU
- J7 pad 1: B_OUT -> C_OUT
- J7 pad 2: B_OUT -> C_OUT
- R2 pad 2: Net-(D1-OUT) -> OUT_MCU
