File: Плата датчиков.kicad_pcb (KiCad board)
At the start: 4 copper layers, 67 x 54.9 mm, 54 parts, among them J1 A, J10 4900, J11 4900, J12 4900, J13 4900, J14 4900, J15 Conn_02x04_Odd_Even, J16 Conn_01x02, J17 Conn_01x02, J2 B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

Commit message: Отправил на проверку в резонит
Parts:
- removed J15: Conn_02x04_Odd_Even, Connector_PinHeader_1.27mm:PinHeader_2x04_P1.27mm_Vertical
- added J18: Conn_02x05_Odd_Even, Connector_PinHeader_1.27mm:PinHeader_2x05_P1.27mm_Vertical, B.Cu at (133.6, 59.6)
- D1: value NSM3012 -> NSM3012B-DSPR
- J16, J17: moved to B.Cu
- turned J16 to 180 degrees
- turned J17 to 180 degrees
Routing:
- net Temp_Coil_A_MCU: track 31.1 -> 31.7 mm
- net B-: vias 128 -> 127
Other:
- board size 67 x 54.9 mm -> 67 x 55.7 mm
