File: Coil_Temperature.kicad_sch (KiCad schematic)
At the start: 14 parts, among them U4 LMV324

Commit message: Собираю документацию
Parts:
- added R15, R19, R20: 9.1k, Resistor_SMD:R_0603_1608Metric_Pad0.98x0.95mm_HandSolder, symbol Device:R_Small
- added R16, R17, R18: 1k, Resistor_SMD:R_0603_1608Metric_Pad0.98x0.95mm_HandSolder, symbol Device:R_Small
- C10, C12, C14: value 100n -> 1u
- R11, R13, R9: value 1.5k -> 15k
Connections:
- net GNDA: now also R16.1, R17.1, R18.1
- net at R12.2, U4.7: now also R15.2; no longer U4.6 (-)
- net at R14.2, U4.8: now also R20.2; no longer U4.9 (-)
- net at R10.2, U4.1: now also R19.2; no longer U4.2 (-)
- new net: R15.1, R16.2, U4.6 (-)
- new net: R17.2, R20.1, U4.9 (-)
- new net: R18.2, R19.1, U4.2 (-)
Other:
- note added: "Температура обмотки B"
- note added: "Температура обмотки С"
