File: Conection_list.kicad_sch (KiCad schematic)
At the start: 0 parts

Commit message: Изменения: добавил папку с отчетностью
Other:
- note added: "A1"
- note added: "Измерительная часть"
- note added: "Соединительная часть"
- note added: "Узел силовой"
