File: Rotary_Position_Sensor.kicad_sch (KiCad schematic)
At the start: 8 parts

Commit message: Добавил все в BOM
Parts:
- D1: value NSM3012 -> NSM3012B-DSPR
Changed lines of the file:
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@@
 			)
 		)
-		(property "Value" "NSM3012"
+		(property "Value" "NSM3012B-DSPR"
 			(at 161.925 93.98 0)
 			(effects
